File: Project/TMC2208/TMC2208.kicad_pcb (KiCad board)
At the start: 2 copper layers, 30.5 x 28.5 mm, 22 parts, among them U2 TMC2208-LA

Commit message: Ki-CAD: TMC2208-WIP2
Parts:
- removed C10: 100nF, Capacitor_Tantalum_SMD:CP_EIA-1608-10_AVX-L
- removed C7, C8: 10uF, Capacitor_Tantalum_SMD:CP_EIA-1608-10_AVX-L
- removed C9: 1uF, Capacitor_Tantalum_SMD:CP_EIA-1608-10_AVX-L
- removed D1: SB120, Diode_SMD:D_MELF-RM10_Universal_Handsoldering
- removed D2: 1N5711, Diode_SMD:D_MELF-RM10_Universal_Handsoldering
- removed R3: R, Resistor_SMD:R_0402_1005Metric
- removed TP1, TP2, TP3, TP4, TP5, TP6: TestPoint, TestPoint:TestPoint_THTPad_1.0x1.0mm_Drill0.5mm
- added J1: Conn_01x08_Pin, Connector_PinHeader_2.54mm:PinHeader_1x08_P2.54mm_Vertical, F.Cu at (151.3, 114.0)
- added J2: Conn_01x08_Pin, Connector_PinHeader_2.54mm:PinHeader_1x08_P2.54mm_Vertical, F.Cu at (151.3, 101.3)
- added R5: 10K, Resistor_SMD:R_0201_0603Metric, F.Cu at (162.4, 111.6)
- added R6: R_Variable, Potentiometer_SMD:Potentiometer_Bourns_TC33X_Vertical, B.Cu at (168.0, 107.2)
- added Vref1: ~, TestPoint:TestPoint_THTPad_1.0x1.0mm_Drill0.5mm, F.Cu at (169.4, 110.4)
- C1: value 22nF -> 100nF; footprint Capacitor_Tantalum_SMD:CP_EIA-1608-10_AVX-L -> Capacitor_SMD:C_0805_2012Metric
- C2: value 1.2uF -> 22nF; footprint Capacitor_Tantalum_SMD:CP_EIA-1608-10_AVX-L -> Capacitor_SMD:C_0805_2012Metric
- C3: footprint Capacitor_THT:CP_Radial_D8.0mm_P2.50mm -> Capacitor_SMD:C_0805_2012Metric
- C4, C6: footprint Capacitor_Tantalum_SMD:CP_EIA-1608-10_AVX-L -> Capacitor_SMD:C_0805_2012Metric
- C5: value 130uF -> 4.7uF; footprint Capacitor_Tantalum_SMD:CP_EIA-1608-10_AVX-L -> Capacitor_SMD:C_0805_2012Metric
- R1, R2: value R -> 0.11E; footprint Resistor_SMD:R_0402_1005Metric -> Resistor_SMD:R_0201_0603Metric
- moved C1 35.0 mm to (152.0, 110.7), turned to 0 degrees
- moved R2 33.8 mm to (166.6, 103.7), turned to 0 degrees
- moved U2 33.4 mm to (160.3, 107.4)
- moved C3 32.9 mm to (166.1, 110.4)
- moved R1 32.4 mm to (159.0, 103.5), turned to 180 degrees
- moved C4 30.7 mm to (151.8, 108.6), turned to 0 degrees
- moved C5 30.1 mm to (155.5, 111.0)
- moved C6 23.5 mm to (151.5, 105.0), turned to -90 degrees
- moved C2 22.7 mm to (154.3, 105.6)
Connections:
- net VCC_IO/2.2D renamed /VIO
- C1 pad 1: Net-(U2-CPI) -> /VM
- C1 pad 2: Net-(U2-CPO) -> Net-(U2-VCP)
- C2 pad 1: 5VOUT/2.3E -> Net-(U2-CPI)
- C2 pad 2: GND -> Net-(U2-CPO)
- C4 pad 1: VS -> /VM
- C5 pad 1: VS -> Net-(U2-5VOUT)
- C6 pad 1: VS -> /VM
- R1 pad 1: Net-(JP2-B) -> Net-(U2-BRB)
- R2 pad 1: Net-(JP3-B) -> Net-(U2-BRA)
- U2 pad 1: Net-(J5-Pin_2) -> /M2B
- U2 pad 10: MS2 -> /MS2
- U2 pad 11: DIAG -> /DIAG
- U2 pad 12: INDEX -> /INDEX
- U2 pad 14: PDN_UART -> /PDN_UART
- U2 pad 16: Net-(J3-Pin_2) -> /STEP
- U2 pad 17: +3.3V -> Net-(U2-VREF)
- U2 pad 19: Net-(J1-Pin_2) -> /DIR
- U2 pad 2: ENN -> /EN
- U2 pad 21: Net-(J5-Pin_4) -> /M2A
- U2 pad 22: VS -> /VM
- U2 pad 23: Net-(JP2-B) -> Net-(U2-BRA)
- U2 pad 24: Net-(J5-Pin_3) -> /M1A
- U2 pad 26: Net-(J5-Pin_1) -> /M1B
- U2 pad 27: Net-(JP3-B) -> Net-(U2-BRB)
- U2 pad 28: VS -> /VM
- U2 pad 8: 5VOUT/2.3E -> Net-(U2-5VOUT)
- U2 pad 9: MS1 -> /MS1
Routing:
- net /VM: track 0.00 -> 28.2 mm, vias 0 -> 3
- net GND: track 0.00 -> 26.6 mm, vias 0 -> 15
- net /VIO: track 0.00 -> 18.9 mm, vias 0 -> 2
- net /EN: track 0.00 -> 15.0 mm, vias 0 -> 1
- net Net-(U2-VREF): track 0.00 -> 11.9 mm, vias 0 -> 1
- net /DIR: track 0.00 -> 10.3 mm, vias 0 -> 1
- net /M2A: track 0.00 -> 8.24 mm, vias 0 -> 1
- net /MS1: track 0.00 -> 6.73 mm
- net /STEP: track 0.00 -> 6.48 mm
- net Net-(U2-VCP): track 0.00 -> 6.20 mm
- net Net-(U2-CPI): track 0.00 -> 5.85 mm
- net /PDN_UART: track 0.00 -> 5.60 mm
- net /M1B: track 0.00 -> 5.37 mm
- net /MS2: track 0.00 -> 5.23 mm
- net /M2B: track 0.00 -> 4.99 mm
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- added copper zone on B.Cu, net GND
- added copper zone on F.Cu, net GND
Other:
- board size 30.5 x 28.5 mm -> 21 x 15.7 mm
