File: Project/TMC2208/TMC2208.kicad_sch (KiCad schematic)
At the start: 34 parts, among them J1 Conn_1X03, J2 Conn_01x02, J3 Conn_01x03, J4 Conn_01x04, J5 Conn_01x08_Pin, J6 Conn_01x08_Pin, U2 TMC2208-LA

Commit message: Ki-CAD: TMC2208-WIP2
Parts:
- removed 10K1: R, Resistor_SMD:R_0402_1005Metric, symbol Device:R
- removed C1: 22nF, Capacitor_Tantalum_SMD:CP_EIA-1608-10_AVX-L, symbol Device:C
- removed C5: 130uF, Capacitor_Tantalum_SMD:CP_EIA-1608-10_AVX-L, symbol Device:C_Polarized
- removed C7, C8: 10uF, Capacitor_Tantalum_SMD:CP_EIA-1608-10_AVX-L, symbol Device:C
- removed C9: 1uF, Capacitor_Tantalum_SMD:CP_EIA-1608-10_AVX-L, symbol Device:C
- removed D1: SB120, Diode_SMD:D_MELF-RM10_Universal_Handsoldering, symbol Diode:SB120
- removed D2: 1N5711, Diode_SMD:D_MELF-RM10_Universal_Handsoldering, symbol Diode:1N5711
- removed J1: Conn_1X03, symbol Connector_Generic:Conn_01x03
- removed J2: Conn_01x02, symbol Connector_Generic:Conn_01x02
- removed J3: Conn_01x03, symbol Connector_Generic:Conn_01x03
- removed J4: Conn_01x04, symbol Connector_Generic:Conn_01x04
- removed J5, J6: Conn_01x08_Pin, symbol Connector:Conn_01x08_Pin
- removed JP1, JP2, JP3: SolderJumper_2_Open, symbol Jumper:SolderJumper_2_Open
- removed R4: 4.7K, symbol Device:R
- removed R6: 10K, symbol Device:R
- removed TP1, TP2, TP3, TP4, TP5, TP6: TestPoint, TestPoint:TestPoint_THTPad_1.0x1.0mm_Drill0.5mm, symbol Connector:TestPoint
- added C2: 22nF, Capacitor_SMD:C_0805_2012Metric, symbol Device:C
- added J1, J2: Conn_01x08_Pin, Connector_PinHeader_2.54mm:PinHeader_1x08_P2.54mm_Vertical, symbol Connector:Conn_01x08_Pin
- added R6: R_Variable, Potentiometer_SMD:Potentiometer_Bourns_TC33X_Vertical, symbol Device:R_Variable
- added Vref1: ~, TestPoint:TestPoint_THTPad_1.0x1.0mm_Drill0.5mm, symbol Connector:TestPoint
- C1: renamed from C10; footprint Capacitor_Tantalum_SMD:CP_EIA-1608-10_AVX-L -> Capacitor_SMD:C_0805_2012Metric
- C3: footprint Capacitor_THT:CP_Radial_D8.0mm_P2.50mm -> Capacitor_SMD:C_0805_2012Metric
- C4, C6: footprint Capacitor_Tantalum_SMD:CP_EIA-1608-10_AVX-L -> Capacitor_SMD:C_0805_2012Metric
- C5: renamed from C2; value 1.2uF -> 4.7uF; footprint Capacitor_Tantalum_SMD:CP_EIA-1608-10_AVX-L -> Capacitor_SMD:C_0805_2012Metric
- R1, R2: value 10K -> 0.11E; footprint Resistor_SMD:R_0402_1005Metric -> Resistor_SMD:R_0201_0603Metric
- R5: value 4.7K -> 10K; footprint (none) -> Resistor_SMD:R_0201_0603Metric
Connections:
- net DIAG: now also J1.4 (Pin_4)
- net DIR: now also J1.8 (Pin_8)
- net GND: now also R5.1, J2.2 (Pin_2), J2.8 (Pin_8), R6.1
- net INDEX: now also J1.5 (Pin_5)
- net M1A: now also U2.24 (OA1), J2.5 (Pin_5); no longer R1.1, U2.23 (BRA)
- net M1B: now also U2.26 (OB1), J2.4 (Pin_4); no longer R2.1, U2.27 (BRB)
- net M2A: now also J2.6 (Pin_6)
- net M2B: now also J2.3 (Pin_3)
- net MS1: now also J1.2 (Pin_2)
- net MS2: now also J1.3 (Pin_3); no longer R5.2
- net PDN_UART: now also R5.2, J1.6 (Pin_6)
- net STEP: now also J1.7 (Pin_7)
- net at U2.4 (CPO): now also C2.2
- net at U2.5 (CPI): now also C2.1
- net +3.3V renamed VIO
- net VIO: now also J2.7 (Pin_7); no longer U2.17 (VREF)
- net +5V renamed VM
- net VM: now also J2.1 (Pin_1); no longer R5.1
- net 5VOUT/2.3E: no longer names the net of C5.1, U2.8 (5VOUT)
- net ENN renamed EN
- net EN: now also J1.1 (Pin_1)
- new net: R1.1, U2.27 (BRB)
- new net: R6.2, U2.17 (VREF), Vref1.1
- new net: R2.1, U2.23 (BRA)
Other:
- note removed: "3.3"
- moved on the sheet: C1, C3, C5, C6, U2
